Commit message: Fix node launch.
Signed-off-by: James Goppert <james.goppert@gmail.com>

File: cubs2_description/urdf/sportcub.urdf.xacro (robot description, xacro)
@@ -10,5 +10,5 @@
         <origin xyz="0 0 -0.1" rpy="0 0 0"/>
         <geometry>
-          <mesh filename="package://fixed_wing_purt/resources/meshes/plane.glb"
+          <mesh filename="package://cubs2_description/meshes/plane.glb"
                 scale="1.0 1.0 1.0"/>
         </geometry>
